File: jeopardy_buzzer_controller.kicad_pcb (KiCad board)
At the start: 2 copper layers, 259.1 x 101.6 mm, 18 parts, among them J1 XLR4_Ground, J2 XLR4_Ground, J3 XLR4_Ground, J4 XLR4_Ground, J5 XLR4_Ground, J6 XLR4_Ground, J7 XLR4_Ground, J8 XLR4_Ground, SW1 RESET, U1 ProMicro

Commit message: Add power LED, enable switch, enable LED
Parts:
- removed REF** (x8): MountingHole_3.2mm_M3_Pad_Via, MountingHole:MountingHole_3.2mm_M3_Pad_Via
- added J11: TO_ENABLE_SWTICH, TerminalBlock_Phoenix:TerminalBlock_Phoenix_MKDS-1,5-2-5.08_1x02_P5.08mm_Horizontal, F.Cu at (63.0, 67.0)
- added J12: TO_ENABLE_LED, TerminalBlock_Phoenix:TerminalBlock_Phoenix_MKDS-1,5-2-5.08_1x02_P5.08mm_Horizontal, F.Cu at (48.6, 67.0)
- added J13: TO_POWER_LED, TerminalBlock_Phoenix:TerminalBlock_Phoenix_MKDS-1,5-2-5.08_1x02_P5.08mm_Horizontal, F.Cu at (35.8, 67.0)
- J1: value XLR4_Ground -> XLR1
- J2: value XLR4_Ground -> XLR2
- J3: value XLR4_Ground -> XLR3
- J4: value XLR4_Ground -> XLR4
- J5: value XLR4_Ground -> XLR5
- J6: value XLR4_Ground -> XLR6
- J7: value XLR4_Ground -> XLR7
- J8: value XLR4_Ground -> XLR8
- moved U1 93.9 mm to (59.5, 47.9)
- moved SW1 80.9 mm to (58.5, 34.0), turned to 180 degrees
- moved J1 77.8 mm to (88.0, 44.4)
- moved J2 75.5 mm to (114.2, 44.4)
- moved J3 73.2 mm to (140.4, 44.4)
- moved J4 71.2 mm to (166.5, 44.4)
- moved J5 69.3 mm to (192.7, 44.4)
- moved J6 67.6 mm to (218.9, 44.4)
- moved J7 66.1 mm to (245.0, 44.4)
- moved J8 64.8 mm to (271.2, 44.4)
Connections:
- SW1 pad 1: Net-(U1-Pad23) -> Net-(SW1-Pad1)
- SW1 pad 2: Net-(U1-Pad22) -> GND
- U1 pad 10: /XLR6 -> unconnected-(U1-Pad10)
- U1 pad 11: /XLR7 -> unconnected-(U1-Pad11)
- U1 pad 12: /XLR8 -> unconnected-(U1-Pad12)
- U1 pad 13: unconnected-(U1-Pad13) -> /XLR8
- U1 pad 14: unconnected-(U1-Pad14) -> /XLR7
- U1 pad 15: unconnected-(U1-Pad15) -> /XLR6
- U1 pad 16: unconnected-(U1-Pad16) -> /XLR5
- U1 pad 17: unconnected-(U1-Pad17) -> /XLR4
- U1 pad 18: unconnected-(U1-Pad18) -> /XLR3
- U1 pad 19: unconnected-(U1-Pad19) -> /XLR2
- U1 pad 20: unconnected-(U1-Pad20) -> /XLR1
- U1 pad 22: Net-(U1-Pad22) -> Net-(SW1-Pad1)
- U1 pad 23: Net-(U1-Pad23) -> GND
- U1 pad 24: unconnected-(U1-Pad24) -> Net-(U1-Pad24)
- U1 pad 3: GND -> unconnected-(U1-Pad3)
- U1 pad 5: /XLR1 -> unconnected-(U1-Pad5)
- U1 pad 6: /XLR2 -> unconnected-(U1-Pad6)
- U1 pad 7: /XLR3 -> Net-(U1-Pad7)
- U1 pad 8: /XLR4 -> Net-(U1-Pad8)
- U1 pad 9: /XLR5 -> unconnected-(U1-Pad9)
Routing:
- net GND: track 439.9 -> 0.00 mm
- net /XLR1: track 126.7 -> 0.00 mm
- net /XLR2: track 103.3 -> 0.00 mm
- net /XLR8: track 102.9 -> 0.00 mm
- net /XLR3: track 74.5 -> 0.00 mm
- net /XLR7: track 73.8 -> 0.00 mm
- net /XLR4: track 54.4 -> 0.00 mm
- net /XLR6: track 50.5 -> 0.00 mm
- net /XLR5: track 39.1 -> 0.00 mm
- net Net-(U1-Pad23): track 14.9 -> 0.00 mm
- net Net-(U1-Pad22): track 14.1 -> 0.00 mm
Other:
- board size 259.1 x 101.6 mm -> 276 x 55 mm
- board text added: "55mm"
- board text added: "Right-angle micro USB"
