File: jeopardy_buzzer_controller.kicad_pcb (KiCad board)
At the start: 2 copper layers, 276 x 55 mm, 13 parts, among them J1 XLR1, J11 TO_ENABLE_SWTICH, J12 TO_ENABLE_LED, J13 TO_POWER_LED, J2 XLR2, J3 XLR3, J4 XLR4, J5 XLR5, J6 XLR6, J7 XLR7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

Commit message: Figured out sensible layout for everything
Parts:
- J11, J12, J13, SW1, U1: moved to B.Cu
- moved J13 286.8 mm to (312.0, 144.0), turned to -90 degrees
- moved SW1 267.7 mm to (309.5, 127.0), turned to -90 degrees
- moved U1 250.8 mm to (293.6, 137.9), turned to -90 degrees
- moved J1 92.3 mm to (80.0, 136.4)
- moved J2 92.3 mm to (106.2, 136.4)
- moved J3 92.3 mm to (132.4, 136.4)
- moved J4 92.3 mm to (158.5, 136.4)
- moved J5 92.3 mm to (184.7, 136.4)
- moved J6 92.3 mm to (210.9, 136.4)
- moved J7 92.3 mm to (237.0, 136.4)
- moved J8 92.3 mm to (263.2, 136.4)
- moved J11 81.0 mm to (62.0, 148.0), turned to 90 degrees
- moved J12 66.4 mm to (62.0, 132.0), turned to 90 degrees
Other:
- board size 276 x 55 mm -> 272 x 38 mm
- board text added: "Clearance needed to (un)plug the USB connector"
- board text added: "Right-angle micro-USB cable"
- board text added: "XLR connectors are on the FRONT of the board. Arduino is on the BACK of the board."
- board text removed: "55mm"
- board text removed: "Right-angle micro USB"

Commit message: Route tracks
Parts:
- U1: value ProMicro -> Arduino Pro Micro
- moved J12 17.0 mm to (63.0, 149.0)
- moved J11 16.0 mm to (63.0, 132.0)
Routing:
- net GND: track 0.00 -> 401.6 mm
- net Net-(J12-Pad2): track 0.00 -> 258.2 mm
- net Net-(J11-Pad2): track 0.00 -> 251.9 mm
- net /XLR1: track 0.00 -> 215.1 mm
- net /XLR2: track 0.00 -> 189.7 mm
- net /XLR3: track 0.00 -> 163.8 mm
- net /XLR4: track 0.00 -> 138.4 mm
- net /XLR5: track 0.00 -> 112.5 mm
- net /XLR6: track 0.00 -> 87.2 mm
- net /XLR7: track 0.00 -> 61.8 mm
- net Net-(J13-Pad1): track 0.00 -> 47.9 mm
- net /XLR8: track 0.00 -> 33.7 mm
- net Net-(SW1-Pad1): track 0.00 -> 30.0 mm
