File: jeopardy_buzzer_controller.kicad_pcb (KiCad board)
At the start: 2 copper layers, 272 x 38 mm, 13 parts, among them J1 XLR1, J11 TO_ENABLE_SWTICH, J12 TO_ENABLE_LED, J13 TO_POWER_LED, J2 XLR2, J3 XLR3, J4 XLR4, J5 XLR5, J6 XLR6, J7 XLR7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

Commit message: Add CERN OHL2-S license
Other:
- board text added: "Copyright 2022 Peter Froud and others. Licensed under CERN-OHL-S v2. Source location: https://github.com/pfroud/jeopardy-buzzer-controller"
- board text added: "Copyright Peter Froud 2022. This source describes Open Hardware and is licensed under the CERN-OHL-S v2. You may redistribute and modify this source and make products using it under the terms of the CERN-OHL-S v2 (https://ohwr.org/cern_ohl_s_v2.txt). This source is distributed WITHOUT ANY EXPRESS OR IMPLIED WARRANTY, INCLUDING OF MERCHANTABILITY, SATISFACTORY QUALITY AND FITNESS FOR A PARTICULAR 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"
Changed lines of the file:
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@@
   (gr_rect (start -50 100) (end 400 155) (layer "User.9") (width 0.1) (fill none))
   (gr_rect (start -78 98) (end 522 157) (layer "User.9") (width 0.1) (fill none))
+  (gr_text "Copyright 2022 Peter Froud and others.\nLicensed under CERN-OHL-S v2.\nSource location: https://github.com/pfroud/jeopardy-buzzer-controller" (at 274 128) (layer "B.SilkS")
+    (effects (font (size 1 1) (thickness 0.15)) (justify left mirror))
+  )
+  (gr_text "Copyright Peter Froud 2022.\n\nThis source describes Open Hardware and is licensed under the CERN-OHL-S v2.\n\nYou may redistribute and modify this source and make products using it under\nthe terms of the CERN-OHL-S v2 (https://ohwr.org/cern_ohl_s_v2.txt).\n\nThis source is distributed WITHOUT ANY EXPRESS OR IMPLIED WARRANTY,\nINCLUDING OF MERCHANTABILITY, SATISFACTORY QUALITY AND FITNESS FOR A\nPARTICULAR PURPOSE. Please see the CERN-OHL-S v2 for applicable conditions. \n\nSource location: https://github.com/pfroud/jeopardy-buzzer-controller" (at 14 193) (layer "User.1")
+    (effects (font (size 1 1) (thickness 0.15)) (justify left))
+  )
   (gr_text "Right-angle micro-USB cable" (at 304 110) (layer "User.2")
     (effects (font (size 1 1) (thickness 0.15)) (justify left))

Commit message: Add title text w/ revision number and date
Other:
- board text added: "Jeopardy buzzer controller"
- board text added: "Revision 1, YYYY-MM-DD"
Changed lines of the file:
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@@
   )
   (paper "USLegal")
+  (title_block
+    (title "Jeopardy buzzer controller")
+  )
   (layers
     (0 "F.Cu" signal)
@@
   (gr_rect (start -50 100) (end 400 155) (layer "User.9") (width 0.1) (fill none))
   (gr_rect (start -78 98) (end 522 157) (layer "User.9") (width 0.1) (fill none))
-  (gr_text "Copyright 2022 Peter Froud and others.\nLicensed under CERN-OHL-S v2.\nSource location: https://github.com/pfroud/jeopardy-buzzer-controller" (at 274 128) (layer "B.SilkS")
+  (gr_text "Jeopardy buzzer controller" (at 280 126) (layer "B.SilkS")
+    (effects (font (size 4 4) (thickness 0.5)) (justify left mirror))
+  )
+  (gr_text "Copyright 2022 Peter Froud and others.\nLicensed under CERN-OHL-S v2.\nSource location: https://github.com/pfroud/jeopardy-buzzer-controller" (at 280 150) (layer "B.SilkS")
     (effects (font (size 1 1) (thickness 0.15)) (justify left mirror))
   )
+  (gr_text "Revision 1, YYYY-MM-DD" (at 189 126) (layer "B.SilkS")
+    (effects (font (size 4 4) (thickness 0.15)) (justify left mirror))
+  )
   (gr_text "Copyright Peter Froud 2022.\n\nThis source describes Open Hardware and is licensed under the CERN-OHL-S v2.\n\nYou may redistribute and modify this source and make products using it under\nthe terms of the CERN-OHL-S v2 (https://ohwr.org/cern_ohl_s_v2.txt).\n\nThis source is distributed WITHOUT ANY EXPRESS OR IMPLIED WARRANTY,\nINCLUDING OF MERCHANTABILITY, SATISFACTORY QUALITY AND FITNESS FOR A\nPARTICULAR PURPOSE. Please see the CERN-OHL-S v2 for applicable conditions. \n\nSource location: https://github.com/pfroud/jeopardy-buzzer-controller" (at 14 193) (layer "User.1")
