File: KiCad_project/jeopardy_buzzer_controller.kicad_pcb (KiCad board)
At the start: 2 copper layers, 272 x 38 mm, 13 parts, among them J1 XLR1, J11 TO_ENABLE_SWTICH, J12 TO_ENABLE_LED, J13 TO_POWER_LED, J2 XLR2, J3 XLR3, J4 XLR4, J5 XLR5, J6 XLR6, J7 XLR7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

Commit message: Vertically center XLR connectors in downspout
Parts:
- J11: value TO_ENABLE_SWTICH -> ENABLE_SW
- J12: value TO_ENABLE_LED -> ENABLE_LED
- J13: value TO_POWER_LED -> PWR_LED
- moved J12 245.0 mm to (308.0, 146.0), turned to -90 degrees
- moved J11 245.0 mm to (308.0, 134.0), turned to -90 degrees
- moved J13 22.4 mm to (308.0, 122.0)
- moved SW1 15.1 mm to (311.5, 112.0), turned to 180 degrees
- moved J1 9.43 mm to (80.0, 127.0)
- moved J2 9.43 mm to (106.2, 127.0)
- moved J3 9.43 mm to (132.4, 127.0)
- moved J4 9.43 mm to (158.5, 127.0)
- moved J5 9.43 mm to (184.7, 127.0)
- moved J6 9.43 mm to (210.9, 127.0)
- moved J7 9.43 mm to (237.0, 127.0)
- moved J8 9.43 mm to (263.2, 127.0)
- moved U1 2.00 mm to (291.6, 137.9)
Connections:
- U1 pad 13: /XLR8 -> /XLR1
- U1 pad 14: /XLR7 -> /XLR2
- U1 pad 15: /XLR6 -> /XLR3
- U1 pad 16: /XLR5 -> /XLR4
- U1 pad 17: /XLR4 -> /XLR5
- U1 pad 18: /XLR3 -> /XLR6
- U1 pad 19: /XLR2 -> /XLR7
- U1 pad 20: /XLR1 -> /XLR8
Routing:
- net Net-(J12-Pad2): track 258.2 -> 12.4 mm
- net Net-(J11-Pad2): track 251.9 -> 8.71 mm
- net GND: track 401.6 -> 364.5 mm
- net Net-(J13-Pad1): track 47.9 -> 24.3 mm
- net /XLR7: track 61.8 -> 56.8 mm
- net /XLR8: track 33.7 -> 28.8 mm
- net Net-(SW1-Pad1): track 30.0 -> 34.6 mm
- net /XLR6: track 87.2 -> 82.9 mm
- net /XLR1: track 215.1 -> 218.9 mm
- net /XLR5: track 112.5 -> 109.9 mm
- net /XLR2: track 189.7 -> 191.8 mm
- net /XLR4: track 138.4 -> 137.6 mm
- net /XLR3: track 163.8 -> 164.4 mm
Other:
- board size 272 x 38 mm -> 250 x 46 mm

Commit message: Add date stamp and generate gerbers!
Other:
- board text added: "Revision 1, 2022-08-22"
- board text removed: "Revision 1, YYYY-MM-DD"
Changed lines of the file:
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@@
       (layerselection 0x00010fc_ffffffff)
       (disableapertmacros false)
-      (usegerberextensions false)
+      (usegerberextensions true)
       (usegerberattributes true)
       (usegerberadvancedattributes true)
@@
       (plotinvisibletext false)
       (sketchpadsonfab false)
-      (subtractmaskfromsilk false)
+      (subtractmaskfromsilk true)
       (outputformat 1)
       (mirror false)
-      (drillshape 1)
+      (drillshape 0)
       (scaleselection 1)
-      (outputdirectory "")
+      (outputdirectory "gerbers/")
     )
   )
@@
     (effects (font (size 1 1) (thickness 0.15)) (justify left mirror))
   )
-  (gr_text "Revision 1, YYYY-MM-DD" (at 173 116) (layer "B.SilkS")
+  (gr_text "Revision 1, 2022-08-22" (at 173 116) (layer "B.SilkS")
     (effects (font (size 5 5) (thickness 0.15)) (justify left mirror))
   )

Commit message: Increase font size and thickness
Other:
- board text added: "Revision 2, YYYY-MM-DD"
- board text removed: "Revision 1, 2022-08-22"
Changed lines of the file:
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@@
   (gr_rect locked (start -50 98) (end 400 157) (layer "User.9") (width 0.1) (fill none))
   (gr_text "Jeopardy buzzer controller" (at 280 116) (layer "B.SilkS")
+    (effects (font (size 5 5) (thickness 1)) (justify left mirror))
+  )
+  (gr_text "Copyright 2022 Peter Froud and others.\nLicensed under CERN-OHL-S v2.\nSource location: https://github.com/pfroud/jeopardy-buzzer-controller" (at 276.86 147.32) (layer "B.SilkS")
+    (effects (font (size 2 2) (thickness 0.2)) (justify left mirror))
+  )
+  (gr_text "Revision 2, YYYY-MM-DD" (at 173 116) (layer "B.SilkS")
     (effects (font (size 5 5) (thickness 0.5)) (justify left mirror))
   )
-  (gr_text "Copyright 2022 Peter Froud and others.\nLicensed under CERN-OHL-S v2.\nSource location: https://github.com/pfroud/jeopardy-buzzer-controller" (at 279 150) (layer "B.SilkS")
-    (effects (font (size 1 1) (thickness 0.15)) (justify left mirror))
-  )
-  (gr_text "Revision 1, 2022-08-22" (at 173 116) (layer "B.SilkS")
-    (effects (font (size 5 5) (thickness 0.15)) (justify left mirror))
-  )
   (gr_text "Copyright Peter Froud 2022.\n\nThis source describes Open Hardware and is licensed under the CERN-OHL-S v2.\n\nYou may redistribute and modify this source and make products using it under\nthe terms of the CERN-OHL-S v2 (https://ohwr.org/cern_ohl_s_v2.txt).\n\nThis source is distributed WITHOUT ANY EXPRESS OR IMPLIED WARRANTY,\nINCLUDING OF MERCHANTABILITY, SATISFACTORY QUALITY AND FITNESS FOR A\nPARTICULAR PURPOSE. Please see the CERN-OHL-S v2 for applicable conditions. \n\nSource location: https://github.com/pfroud/jeopardy-buzzer-controller" (at 14 193) (layer "User.1")

Commit message: Add custom XLR footprint with bigger holes
Adding a modified version of the "Jack_XLR_Neutrik_NC4MBV_Vertical"
footprint included in the KiCad "Connector_Audio" library.

The NC4MBV footprint included with KiCad uses hole sizes specified by
Neutrik here: https://www.neutrik.com/en/product/nc4mbv-1

Pins 1 through 4 are cylindrical, with a double-taper on the tip
and then a shoulder. The ground pin is rectangular with a shoulder only.

The hole sizes specified by Neutrik are for having the pin shoulders
sit on the PCB. They work perfectly for that - the jack can be
pushed into the PCB with a little force, then the pin shoulders hit the
PCB with a satisfying click, and the jack stays held in the PCB by
friction.

But, I want the full diameter of the pins to go through the holes and
the black plastic housing to sit on the PCB.

Changes to the footprint:

* For pads 1 through 4: increase hole size from 1.6mm to 1.95mm.
    * Lead diameter measured with calipers is 1.75mm.
    * Add 0.20mm clearance per https://klc.kicad.org/footprint/f7/f7.6/.

* For pads 1 and 4 only: increase pad size from 3.4mm to 4mm.
     * The PCB will be supported by the XLR connectors so I want a
       strong solder connection.
     * Can't increase pad size on pads 2 and 3 because they're already
       pretty close to each other.

* For the G pad: change shape from circle to oval.
    * The pin is rectangular. The size measured with calipers is
      2.00mm width and 0.50mm height.
    * Per https://klc.kicad.org/footprint/f7/f7.7/:
        * Set the hole height to be the pin height plus 0.20mm.
          0.5mm + 0.2mm = 0.7mm.
        * Set the hole width to be the pin width plus the hole height.
          2mm + 0.7mm = 2.7mm.
    * Make the pad 2mm larger than the hole for strong solder.

* Add more ref texts above and below the pads on both front and back
  silkscreen. Helpful for keeping track of where you are when soldering
  under a microscope.

* TODO: fix silkscreen arc intersecting t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
Parts:
- XLR1: renamed from J1; footprint Connector_Audio:Jack_XLR_Neutrik_NC4MBV_Vertical -> custom_xlr_footprint:Jack_XLR_Neutrik_NC4MBV_Vertical_with_bigger_holes
- XLR2: renamed from J2; footprint Connector_Audio:Jack_XLR_Neutrik_NC4MBV_Vertical -> custom_xlr_footprint:Jack_XLR_Neutrik_NC4MBV_Vertical_with_bigger_holes
- XLR3: renamed from J3; footprint Connector_Audio:Jack_XLR_Neutrik_NC4MBV_Vertical -> custom_xlr_footprint:Jack_XLR_Neutrik_NC4MBV_Vertical_with_bigger_holes
- XLR4: renamed from J4; footprint Connector_Audio:Jack_XLR_Neutrik_NC4MBV_Vertical -> custom_xlr_footprint:Jack_XLR_Neutrik_NC4MBV_Vertical_with_bigger_holes
- XLR5: renamed from J5; footprint Connector_Audio:Jack_XLR_Neutrik_NC4MBV_Vertical -> custom_xlr_footprint:Jack_XLR_Neutrik_NC4MBV_Vertical_with_bigger_holes
- XLR6: renamed from J6; footprint Connector_Audio:Jack_XLR_Neutrik_NC4MBV_Vertical -> custom_xlr_footprint:Jack_XLR_Neutrik_NC4MBV_Vertical_with_bigger_holes
- XLR7: renamed from J7; footprint Connector_Audio:Jack_XLR_Neutrik_NC4MBV_Vertical -> custom_xlr_footprint:Jack_XLR_Neutrik_NC4MBV_Vertical_with_bigger_holes
- XLR8: renamed from J8; footprint Connector_Audio:Jack_XLR_Neutrik_NC4MBV_Vertical -> custom_xlr_footprint:Jack_XLR_Neutrik_NC4MBV_Vertical_with_bigger_holes
